Commit message: model&world init and set sensors

File: src/petbot_description/urdf/petbot.gazebo.xacro (robot description, xacro)
@@ -1,5 +1,4 @@
 <?xml version="1.0"?>
 <robot xmlns:xacro="http://www.ros.org/wiki/xacro">
-  <!-- 颜色材质 -->
   <gazebo reference="base_link">
     <material>Gazebo/Blue</material>
@@ -7,6 +6,6 @@
   <gazebo reference="left_wheel_link">
     <material>Gazebo/Black</material>
-    <mu1>1.5</mu1>
-    <mu2>1.5</mu2>
+    <mu1>2.5</mu1>
+    <mu2>2.5</mu2>
     <kp>1000000.0</kp>
     <kd>100.0</kd>
@@ -16,6 +15,6 @@
   <gazebo reference="right_wheel_link">
     <material>Gazebo/Black</material>
-    <mu1>1.5</mu1>
-    <mu2>1.5</mu2>
+    <mu1>2.5</mu1>
+    <mu2>2.5</mu2>
     <kp>1000000.0</kp>
     <kd>100.0</kd>
@@ -31,41 +30,4 @@
     <minDepth>0.001</minDepth>
   </gazebo>
-  <gazebo reference="laser_link">
-    <material>Gazebo/Orange</material>
-    <sensor name="lidar" type="ray">
-      <always_on>true</always_on>
-      <visualize>true</visualize>
-      <update_rate>10</update_rate>
-      <pose>0 0 0 0 0 0</pose>
-      <ray>
-        <scan>
-          <horizontal>
-            <samples>360</samples>
-            <resolution>1</resolution>
-            <min_angle>-3.14159</min_angle>
-            <max_angle>3.14159</max_angle>
-          </horizontal>
-        </scan>
-        <range>
-          <min>0.12</min>
-          <max>12.0</max>
-          <resolution>0.01</resolution>
-        </range>
-        <noise>
-          <type>gaussian</type>
-          <mean>0.0</mean>
-          <stddev>0.01</stddev>
-        </noise>
-      </ray>
-      <plugin name="gazebo_ros_laser" filename="libgazebo_ros_ray_sensor.so">
-        <ros>
-          <remapping>~/out:=scan</remapping>
-        </ros>
-        <output_type>sensor_msgs/LaserScan</output_type>
-        <frame_name>laser_link</frame_name>
-      </plugin>
-    </sensor>
-  </gazebo>
-  <!-- 差速驱动插件 -->
   <gazebo>
     <plugin name="gazebo_ros_diff_drive" filename="libgazebo_ros_diff_drive.so">
@@ -77,7 +39,8 @@
       <right_joint>right_wheel_joint</right_joint>
       <wheel_separation>0.22</wheel_separation>
-      <wheel_diameter>0.10</wheel_diameter>
-      <max_wheel_torque>20</max_wheel_torque>
-      <max_wheel_acceleration>2.0</max_wheel_acceleration>
+      <wheel_diameter>0.08</wheel_diameter>
+      <!-- 扭矩/加速度收紧，避免瞬时冲击掀翻（峰值速度仍由 cmd_vel 限幅） -->
+      <max_wheel_torque>12</max_wheel_torque>
+      <max_wheel_acceleration>18.0</max_wheel_acceleration>
       <command_topic>cmd_vel</command_topic>
       <publish_odom>true</publish_odom>
@@ -88,5 +51,4 @@
       <robot_base_frame>base_footprint</robot_base_frame>
     </plugin>
-    <!-- 发布关节状态，供 robot_state_publisher 更新轮子 TF -->
     <plugin name="gazebo_ros_joint_state_publisher"
             filename="libgazebo_ros_joint_state_publisher.so">

File: src/petbot_description/urdf/petbot.urdf.xacro (robot description, xacro)
@@ -2,22 +2,26 @@
 <robot xmlns:xacro="http://www.ros.org/wiki/xacro" name="petbot">
   <!-- ===================== 几何参数 ===================== -->
-  <xacro:property name="base_length" value="0.28"/>
-  <xacro:property name="base_width" value="0.20"/>
-  <xacro:property name="base_height" value="0.08"/>
-  <xacro:property name="base_mass" value="8.0"/>
-  <xacro:property name="wheel_radius" value="0.05"/>
-  <xacro:property name="wheel_width" value="0.04"/>
-  <xacro:property name="wheel_mass" value="0.8"/>
+  <!-- 主体：前后长 20cm × 宽 15cm × 高 15cm；质量加大且重心压低防翻 -->
+  <xacro:property name="base_length" value="0.20"/>
+  <xacro:property name="base_width" value="0.15"/>
+  <xacro:property name="base_height" value="0.15"/>
+  <xacro:property name="base_mass" value="15.0"/>
+  <xacro:property name="wheel_radius" value="0.04"/>
+  <xacro:property name="wheel_width" value="0.03"/>
+  <xacro:property name="wheel_mass" value="0.5"/>
+  <!-- 支撑三角形尽量铺开 -->
   <xacro:property name="wheel_separation" value="0.22"/>
-  <!-- 驱动轮略靠后，提高稳定性 -->
-  <xacro:property name="wheel_x_offset" value="-0.02"/>
+  <xacro:property name="wheel_x_offset" value="-0.08"/>
   <xacro:property name="base_z" value="${wheel_radius}"/>
-  <xacro:property name="caster_radius" value="0.025"/>
-  <xacro:property name="caster_mass" value="0.15"/>
-  <xacro:property name="caster_x" value="0.10"/>
-  <xacro:property name="lidar_radius" value="0.035"/>
-  <xacro:property name="lidar_height" value="0.04"/>
-  <xacro:property name="lidar_mass" value="0.15"/>
-  <xacro:property name="lidar_z" value="${base_height / 2 + lidar_height / 2 + 0.01}"/>
+  <!-- 视觉厢体上移；惯性中心贴近轮轴高度，降低翻车力矩 -->
+  <xacro:property name="base_z_offset" value="${base_height/2 - 0.02}"/>
+  <xacro:property name="base_com_z" value="0.015"/>
+  <xacro:property name="caster_radius" value="0.02"/>
+  <xacro:property name="caster_mass" value="0.12"/>
+  <xacro:property name="caster_x" value="${base_length/2 - 0.005}"/>
+  <!-- Nebula280MIPI：头部（前面中间靠上），轻微上仰 -->
+  <xacro:property name="nebula280_x" value="${base_length/2 - 0.01}"/>
+  <xacro:property name="nebula280_z" value="${base_z_offset + base_height/2 - 0.008}"/>
+  <xacro:property name="nebula280_pitch" value="0.10"/>
   <xacro:macro name="box_inertia" params="m l w h">
     <inertia
@@ -41,5 +45,4 @@
   <material name="black"><color rgba="0.10 0.10 0.10 1.0"/></material>
   <material name="gray"><color rgba="0.55 0.55 0.55 1.0"/></material>
-  <material name="orange"><color rgba="0.95 0.55 0.10 1.0"/></material>
   <link name="base_footprint"/>
   <joint name="base_joint" type="fixed">
@@ -50,5 +53,5 @@
   <link name="base_link">
     <visual>
-      <origin xyz="0 0 0" rpy="0 0 0"/>
+      <origin xyz="0 0 ${base_z_offset}" rpy="0 0 0"/>
       <geometry>
         <box size="${base_length} ${base_width} ${base_height}"/>
@@ -57,5 +60,5 @@
     </visual>
     <collision>
-      <origin xyz="0 0 0" rpy="0 0 0"/>
+      <origin xyz="0 0 ${base_z_offset}" rpy="0 0 0"/>
       <geometry>
         <box size="${base_length} ${base_width} ${base_height}"/>
@@ -63,8 +66,8 @@
     </collision>
     <inertial>
-      <!-- COM 略压低，减少倾覆 -->
-      <origin xyz="0 0 -0.01" rpy="0 0 0"/>
+      <!-- 重心靠近轮轴高度，视觉仍用较高厢体 -->
+      <origin xyz="0 0 ${base_com_z}" rpy="0 0 0"/>
       <mass value="${base_mass}"/>
-      <xacro:box_inertia m="${base_mass}" l="${base_length}" w="${base_width}" h="${base_height}"/>
+      <xacro:box_inertia m="${base_mass}" l="${base_length}" w="${base_width}" h="${base_height * 0.35}"/>
     </inertial>
   </link>
@@ -78,5 +81,4 @@
         <material name="black"/>
       </visual>
-      <!-- 球体碰撞接触更稳 -->
       <collision>
         <origin xyz="0 0 0" rpy="0 0 0"/>
@@ -94,5 +96,4 @@
       <parent link="base_link"/>
       <child link="${prefix}_wheel_link"/>
-      <!-- 轮心与 base_link 同高（= wheel_radius），使轮缘触地 -->
       <origin xyz="${wheel_x_offset} ${y_reflect * wheel_separation / 2} 0" rpy="0 0 0"/>
       <axis xyz="0 1 0"/>
@@ -127,29 +128,14 @@
     <origin xyz="${caster_x} 0 ${-base_z + caster_radius}" rpy="0 0 0"/>
   </joint>
-  <link name="laser_link">
-    <visual>
-      <origin xyz="0 0 0" rpy="0 0 0"/>
-      <geometry>
-        <cylinder radius="${lidar_radius}" length="${lidar_height}"/>
-      </geometry>
-      <material name="orange"/>
-    </visual>
-    <collision>
-      <origin xyz="0 0 0" rpy="0 0 0"/>
-      <geometry>
-        <cylinder radius="${lidar_radius}" length="${lidar_height}"/>
-      </geometry>
-    </collision>
-    <inertial>
-      <origin xyz="0 0 0" rpy="0 0 0"/>
-      <mass value="${lidar_mass}"/>
-      <xacro:cylinder_inertia m="${lidar_mass}" r="${lidar_radius}" h="${lidar_height}"/>
-    </inertial>
-  </link>
-  <joint name="laser_joint" type="fixed">
-    <parent link="base_link"/>
-    <child link="laser_link"/>
-    <origin xyz="0.04 0 ${lidar_z}" rpy="0 0 0"/>
-  </joint>
+  <!-- 传感器：六轴 IMU + Nebula280MIPI -->
+  <xacro:include filename="$(find petbot_description)/urdf/sensors/imu_6axis.urdf.xacro"/>
+  <xacro:imu_6axis parent="base_link">
+    <!-- 靠近底盘几何中心、略高于厢体底板 -->
+    <origin xyz="0 0 ${base_z_offset - base_height/2 + 0.01}" rpy="0 0 0"/>
+  </xacro:imu_6axis>
+  <xacro:include filename="$(find petbot_description)/urdf/sensors/nebula280_mipi.urdf.xacro"/>
+  <xacro:nebula280_mipi parent="base_link">
+    <origin xyz="${nebula280_x} 0 ${nebula280_z}" rpy="0 ${nebula280_pitch} 0"/>
+  </xacro:nebula280_mipi>
   <xacro:include filename="$(find petbot_description)/urdf/petbot.gazebo.xacro"/>
 </robot>
